File: Eagle/Boards/Training Program/UnoMotorShieldsW2016/Cristian/MotorDriver2.brd (EAGLE design)
At the start: 62.5 x 66 mm, 26 parts, among them J1 ARDUINO_UNO_R3

Commit message: compiled 1st board for fabrication
Parts:
- added E$22: (no value), ISCTRainingProgram:1X04
Connections:
- new net S$105: J1.D10
Routing:
- net S$101: track 0.00 -> 22.7 mm
- net S$102: track 0.00 -> 13.3 mm
- net S$35: track 0.76 -> 13.4 mm
- net S$107: track 0.00 -> 11.3 mm, vias 0 -> 1
- net S$97: track 0.00 -> 9.45 mm, vias 0 -> 2
- net S$105: track 0.00 -> 8.09 mm
- net S$106: track 0.00 -> 7.84 mm
- net S$4: track 52.9 -> 45.4 mm, vias 3 -> 2
- net S$96: track 0.00 -> 6.65 mm
- net S$95: track 0.00 -> 5.00 mm, vias 0 -> 1
- net S$103: track 0.00 -> 4.50 mm
- net S$98: track 0.00 -> 4.27 mm
- net S$104: track 0.00 -> 1.71 mm
- net S$100: track 0.00 -> 1.50 mm, vias 0 -> 1
- net S$94: track 7.62 -> 6.50 mm
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Other:
- board text added: "power diode"
- board text removed: "GND"
