File: Eagle/Boards/Training Program/UnoMotorShieldsW2016/Hashim/FirstSchematic.brd (EAGLE design)
At the start: 100 x 80 mm, 5 parts, among them J1 ARDUINO_UNO_R3

Commit message: compiled 1st board for fabrication
Parts:
- added E$1: (no value), ISCTRainingProgram:5.5-2.5-BARRELCONNECTOR
Routing:
- net S$19: track 0.00 -> 25.1 mm, vias 0 -> 1
- net S$1: track 0.00 -> 20.4 mm
- net S$2: track 0.00 -> 10.0 mm
- net S$4: track 0.00 -> 5.61 mm, vias 0 -> 1
- net S$9: track 0.00 -> 5.08 mm, vias 0 -> 1
- net S$8: track 0.00 -> 5.08 mm, vias 0 -> 1
- net S$10: track 0.00 -> 5.08 mm, vias 0 -> 1
- net S$6: track 0.00 -> 5.08 mm, vias 0 -> 1
- net S$5: track 0.00 -> 5.08 mm, vias 0 -> 1
- net S$14: track 0.00 -> 5.08 mm, vias 0 -> 1
- net S$20: track 0.00 -> 4.58 mm
- net S$3: track 0.00 -> 4.34 mm, vias 0 -> 1
- net S$7: track 0.00 -> 3.81 mm, vias 0 -> 1
- net S$18: track 0.00 -> 3.59 mm, vias 0 -> 1
- net S$13: track 0.00 -> 3.07 mm, vias 0 -> 1
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Other:
- board size 100 x 80 mm -> 56 x 66 mm
Changed lines of the file:
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@@
 <?xml version="1.0" encoding="utf-8"?>
 <!DOCTYPE eagle SYSTEM "eagle.dtd">
-<eagle version="7.2.0">
+<eagle version="7.5.0">
 <drawing>
 <settings>
@@
 <setting verticaltext="up"/>
 </settings>
-<grid distance="0.1" unitdist="mm" unit="mm" style="lines" multiple="1" display="no" altdistance="0.025" altunitdist="inch" altunit="inch"/>
+<grid distance="2" unitdist="mm" unit="mm" style="lines" multiple="1" display="no" altdistance="0.025" altunitdist="inch" altunit="inch"/>
 <layers>
 <layer number="1" name="Top" color="4" fill="1" visible="yes" active="yes"/>
+<layer number="2" name="Route2" color="1" fill="3" visible="yes" active="yes"/>
+<layer number="3" name="Route3" color="4" fill="3" visible="yes" active="yes"/>
+<layer number="4" name="Route4" color="1" fill="4" visible="yes" active="yes"/>
+<layer number="5" name="Route5" color="4" fill="4" visible="yes" active="yes"/>
+<layer number="6" name="Route6" color="1" fill="8" visible="yes" active="yes"/>
+<layer number="7" name="Route7" color="4" fill="8" visible="yes" active="yes"/>
+<layer number="8" name="Route8" color="1" fill="2" visible="yes" active="yes"/>
+<layer number="9" name="Route9" color="4" fill="2" visible="yes" active="yes"/>
+<layer number="10" name="Route10" color="1" fill="7" visible="yes" active="yes"/>
+<layer number="11" name="Route11" color="4" fill="7" visible="yes" active="yes"/>
+<layer number="12" name="Route12" color="1" fill="5" visible="yes" active="yes"/>
+<layer number="13" name="Route13" color="4" fill="5" visible="yes" active="yes"/>
+<layer number="14" name="Route14" color="1" fill="6" visible="yes" active="yes"/>
+<layer number="15" name="Route15" color="4" fill="6" visible="yes" active="yes"/>
 <layer number="16" name="Bottom" color="1" fill="1" visible="yes" active="yes"/>
 <layer number="17" name="Pads" color="2" fill="1" visible="yes" active="yes"/>
@@
 <board>
 <plain>
-<wire x1="64" y1="0" x2="100" y2="0" width="0" layer="20"/>
-<wire x1="100" y1="0" x2="100" y2="80" width="0" layer="20"/>
-<wire x1="100" y1="80" x2="0" y2="80" width="0" layer="20"/>
-<wire x1="0" y1="80" x2="0" y2="66" width="0" layer="20"/>
-<wire x1="0" y1="0" x2="0" y2="66" width="0.4064" layer="20"/>
-<wire x1="0" y1="66" x2="64" y2="66" width="0.4064" layer="20"/>
-<wire x1="64" y1="66" x2="64" y2="0" width="0.4064" layer="20"/>
-<wire x1="64" y1="0" x2="0" y2="0" width="0.4064" layer="20"/>
-<text x="23.4" y="59.1" size="1.778" layer="1">Hashim</text>
+<text x="17.05" y="55.29" size="3.81" layer="1">Hashim</text>
+<wire x1="4" y1="0" x2="4" y2="66" width="1.9304" layer="20"/>
+<wire x1="4" y1="66" x2="60" y2="66" width="1.9304" layer="20"/>
+<wire x1="60" y1="66" x2="60" y2="0" width="1.9304" layer="20"/>
+<wire x1="60" y1="0" x2="4" y2="0" width="1.9304" layer="20"/>
 </plain>
 <attributes>
@@
 <attribute name="OC_FARNELL" value="unknown" x="14.88" y="50.96" size="1.778" layer="27" display="off"/>
 </element>
+<element name="E$1" library="ISCTRainingProgram" package="5.5-2.5-BARRELCONNECTOR" value="" x="42.7" y="58.1" rot="R180"/>
 </elements>
 <signals>
@@
 <contactref element="U$1" pad="P6"/>
 <wire x1="33.54" y1="49.69" x2="33.54" y2="44.16" width="0.8128" layer="1"/>
-<wire x1="33.54" y1="44.16" x2="39.3" y2="38.4" width="0.8128" layer="1"/>
-<via x="39.3" y="38.4" extent="1-16" drill="1" shape="square"/>
-<wire x1="39.3" y1="38.4" x2="38.5" y2="32.4" width="0.8128" layer="16"/>
+<wire x1="33.54" y1="44.16" x2="39.3" y2="39.035" width="0.8128" layer="1"/>
+<via x="39.3" y="39.035" extent="1-16" drill="1" shape="square"/>
+<wire x1="39.3" y1="39.035" x2="38.5" y2="32.4" width="0.8128" layer="16"/>
 <wire x1="38.5" y1="32.4" x2="36.7" y2="29.3" width="0.8128" layer="16"/>
 <via x="36.7" y="29.3" extent="1-16" drill="1" shape="square"/>
@@
 <wire x1="34.86" y1="19.75" x2="34.31" y2="19.2" width="0.8128" layer="1"/>
 </signal>
+<signal name="S$1">
+<wire x1="45.9" y1="57.9" x2="48.2" y2="57.9" width="1.27" layer="16"/>
+<wire x1="48.2" y1="57.9" x2="51.7" y2="54.4" width="1.27" layer="16"/>
+<wire x1="51.7" y1="54.4" x2="51.7" y2="45.66" width="1.27" layer="16"/>
+<wire x1="51.7" y1="45.66" x2="55.8" y2="44.1" width="1.27" layer="16"/>
+</signal>
+<signal name="S$2">
+<wire x1="39.8" y1="58.1" x2="39.8" y2="57.8" width="1.27" layer="16"/>
+<wire x1="39.8" y1="57.8" x2="44.7" y2="52.9" width="1.27" layer="16"/>
+<wire x1="44.7" y1="52.9" x2="44.7" y2="50.4" width="1.27" layer="16"/>
+<wire x1="44.7" y1="50.4" x2="44.9" y2="50.2" width="1.27" layer="16"/>
+</signal>
+<signal name="S$3">
+<wire x1="17.78" y1="49.53" x2="20.32" y2="49.53" width="1.27" layer="16"/>
+<wire x1="20.32" y1="49.53" x2="21.59" y2="48.26" width="1.27" layer="16"/>
+<via x="21.59" y="48.26" extent="1-16" drill="0.6"/>
+</signal>
+<signal name="S$4">
+<wire x1="12.7" y1="49.53" x2="12.7" y2="48.26" width="1.27" layer="16"/>
+<wire x1="12.7" y1="48.26" x2="13.97" y2="46.99" width="1.27" layer="16"/>
+<wire x1="13.97" y1="46.99" x2="13.97" y2="44.45" width="1.27" layer="16"/>
+<via x="13.97" y="44.45" extent="1-16" drill="0.6"/>
+</signal>
+<signal name="S$5">
+<wire x1="29.21" y1="49.53" x2="29.21" y2="44.45" width="1.27" layer="16"/>
+<via x="29.21" y="44.45" extent="1-16" drill="0.6"/>
+</signal>
+<signal name="S$6">
+<wire x1="34.29" y1="49.53" x2="34.29" y2="44.45" width="1.27" layer="16"/>
+<via x="34.29" y="44.45" extent="1-16" drill="0.6"/>
+</signal>
+<signal name="S$8">
+<wire x1="26.67" y1="36.83" x2="24.13" y2="36.83" width="0.8128" layer="16"/>
+<via x="24.13" y="36.83" extent="1-16" drill="0.6"/>
+<wire x1="26.67" y1="36.83" x2="24.13" y2="36.83" width="0.8128" layer="1"/>
+</signal>
+<signal name="S$9">
+<wire x1="26.67" y1="34.29" x2="24.13" y2="34.29" width="0.8128" layer="16"/>
+<via x="24.13" y="34.29" extent="1-16" drill="0.6"/>
+<wire x1="26.67" y1="34.29" x2="24.13" y2="34.29" width="0.8128" layer="1"/>
+</signal>
+<signal name="S$10">
+<wire x1="26.67" y1="29.21" x2="24.13" y2="29.21" width="0.8128" layer="16"/>
+<via x="24.13" y="29.21" extent="1-16" drill="0.6"/>
+<wire x1="24.13" y1="29.21" x2="26.67" y2="29.21" width="0.8128" layer="1"/>
+</signal>
+<signal name="S$11">
+<wire x1="26.67" y1="24.13" x2="24.13" y2="24.13" width="0.8128" layer="16"/>
+<via x="24.13" y="24.13" extent="1-16" drill="0.6"/>
+</signal>
+<signal name="S$12">
+<wire x1="26.67" y1="21.59" x2="24.13" y2="21.59" width="0.8128" layer="16"/>
+</signal>
+<signal name="S$13">
+<wire x1="26.67" y1="19.05" x2="25.4" y2="17.78" width="0.8128" layer="16"/>
+<via x="25.4" y="17.78" extent="1-16" drill="0.6"/>
+<wire x1="25.4" y1="17.78" x2="25.4" y2="19.05" width="0.8128" layer="1"/>
+</signal>
+<signal name="S$14">
+<wire x1="34.29" y1="19.05" x2="36.83" y2="19.05" width="0.8128" layer="16"/>
+<via x="36.83" y="19.05" extent="1-16" drill="0.6"/>
+<wire x1="34.29" y1="19.05" x2="36.83" y2="19.05" width="0.8128" layer="1"/>
+</signal>
+<signal name="S$15">
+<wire x1="34.29" y1="21.59" x2="33.02" y2="21.59" width="0.8128" layer="16"/>
+<wire x1="33.02" y1="21.59" x2="31.75" y2="20.32" width="0.8128" layer="16"/>
+<via x="31.75" y="20.32" extent="1-16" drill="0.6"/>
+</signal>
+<signal name="S$16">
+<wire x1="34.29" y1="24.13" x2="35.56" y2="25.4" width="0.8128" layer="16"/>
+</signal>
+<signal name="S$17">
+<wire x1="34.29" y1="31.75" x2="35.56" y2="31.75" width="0.8128" layer="16"/>
+<wire x1="35.56" y1="31.75" x2="36.83" y2="30.48" width="0.8128" layer="16"/>
+</signal>
+<signal name="S$18">
+<wire x1="35.56" y1="34.29" x2="36.83" y2="33.02" width="0.8128" layer="16"/>
+<via x="36.83" y="33.02" extent="1-16" drill="0.6"/>
+<wire x1="35.56" y1="34.29" x2="36.83" y2="33.02" width="0.8128" layer="1"/>
+</signal>
+<signal name="S$19">
+<wire x1="35.56" y1="36.83" x2="36.83" y2="36.83" width="0.8128" layer="16"/>
+<via x="36.83" y="36.83" extent="1-16" drill="0.6"/>
+<wire x1="35.56" y1="36.83" x2="36.83" y2="36.83" width="0.8128" layer="1"/>
+<wire x1="36.83" y1="36.83" x2="39.37" y2="36.83" width="0.8128" layer="1"/>
+<wire x1="39.37" y1="36.83" x2="41.275" y2="36.83" width="0.8128" layer="1"/>
+<wire x1="41.275" y1="36.83" x2="48.26" y2="43.815" width="0.8128" layer="1"/>
+<wire x1="48.26" y1="43.815" x2="48.26" y2="49.53" width="0.8128" layer="1"/>
+<wire x1="34.29" y1="36.83" x2="36.83" y2="36.83" width="0.8128" layer="1"/>
+</signal>
+<signal name="S$20">
+<wire x1="55.88" y1="43.815" x2="52.07" y2="46.355" width="0.8128" layer="1"/>
+</signal>
+<signal name="S$21">
+<via x="52.07" y="45.72" extent="1-16" drill="0.6"/>
+</signal>
+<signal name="S$7">
+<via x="48.26" y="45.72" extent="1-16" drill="0.6"/>
+<wire x1="48.26" y1="45.72" x2="48.26" y2="49.53" width="0.8128" layer="16"/>
+</signal>
 </signals>
