File: Eagle/Boards/Training Program/rPiMotorShield (do last).brd (EAGLE design)
At the start: 88.9 x 127 mm, 29 parts

Commit message: added default board
Routing:
- added copper zone on layer 16, net S$92
- added copper zone on layer 1, net S$93
Changed lines of the file:
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@@
 <setting verticaltext="up"/>
 </settings>
-<grid distance="1" unitdist="mm" unit="mm" style="lines" multiple="1" display="no" altdistance="0.127" altunitdist="mm" altunit="mm"/>
+<grid distance="0.5" unitdist="inch" unit="inch" style="lines" multiple="1" display="no" altdistance="0.127" altunitdist="mm" altunit="mm"/>
 <layers>
 <layer number="1" name="Top" color="4" fill="1" visible="yes" active="yes"/>
@@
 <wire x1="76.2" y1="38.1" x2="78.74" y2="40.64" width="1.4224" layer="1"/>
 <wire x1="78.74" y1="40.64" x2="77.47" y2="41.91" width="1.4224" layer="1"/>
+<via x="76.2" y="115.57" extent="1-16" drill="1"/>
+<wire x1="76.2" y1="109.22" x2="76.2" y2="115.57" width="1.4224" layer="16"/>
+<wire x1="76.2" y1="115.57" x2="76.2" y2="109.22" width="1.4224" layer="1"/>
 <wire x1="76.2" y1="92.71" x2="76.2" y2="92.71" width="0" layer="19" extent="1-16"/>
 <wire x1="76.2" y1="58.42" x2="76.2" y2="58.42" width="0" layer="19" extent="1-16"/>
 <wire x1="76.2" y1="19.05" x2="76.2" y2="19.05" width="0" layer="19" extent="1-16"/>
-<via x="76.2" y="115.57" extent="1-16" drill="1"/>
-<wire x1="76.2" y1="109.22" x2="76.2" y2="115.57" width="1.4224" layer="16"/>
-<wire x1="76.2" y1="115.57" x2="76.2" y2="109.22" width="1.4224" layer="1"/>
 </signal>
 <signal name="S$33">
@@
 <wire x1="62.738" y1="3.175" x2="62.738" y2="2.286" width="1.4224" layer="1"/>
 <wire x1="62.738" y1="2.286" x2="62.103" y2="1.651" width="1.4224" layer="1"/>
-<wire x1="62.103" y1="1.651" x2="16.129" y2="1.651" width="0" layer="19" extent="1-16"/>
 <wire x1="16.51" y1="1.27" x2="15.24" y2="2.54" width="1.016" layer="1"/>
 <wire x1="15.24" y1="2.54" x2="16.51" y2="1.27" width="1.016" layer="16"/>
@@
 <wire x1="52.578" y1="1.27" x2="32.258" y2="1.27" width="1.016" layer="1"/>
 <wire x1="32.258" y1="1.27" x2="16.51" y2="1.27" width="1.016" layer="1"/>
-<wire x1="16.51" y1="1.27" x2="16.129" y2="1.651" width="0" layer="19" extent="1-16"/>
 <wire x1="32.258" y1="3.302" x2="32.258" y2="1.27" width="1.016" layer="16"/>
 <wire x1="32.258" y1="1.27" x2="32.258" y2="3.302" width="1.016" layer="1"/>
 <wire x1="52.578" y1="3.429" x2="52.578" y2="1.27" width="1.016" layer="1"/>
+<wire x1="62.865" y1="3.175" x2="62.738" y2="3.175" width="0" layer="19" extent="1-16"/>
+<wire x1="62.865" y1="3.175" x2="62.865" y2="3.175" width="0" layer="19" extent="1-16"/>
 </signal>
 <signal name="S$68">
 <wire x1="27.178" y1="3.302" x2="27.178" y2="1.397" width="1.016" layer="1"/>
 <wire x1="27.178" y1="1.397" x2="27.178" y2="3.302" width="1.016" layer="16"/>
+<wire x1="27.178" y1="1.397" x2="27.178" y2="1.397" width="0" layer="19" extent="1-16"/>
 </signal>
 <signal name="S$79">
@@
 <wire x1="70.612" y1="24.638" x2="69.977" y2="25.273" width="0.6096" layer="16"/>
 </signal>
+<signal name="S$92">
+<polygon width="1.016" layer="16" spacing="1.016" isolate="1.016">
+<vertex x="0" y="127"/>
+<vertex x="88.9" y="127"/>
+<vertex x="88.9" y="0"/>
+<vertex x="0" y="0"/>
+</polygon>
+</signal>
+<signal name="S$93">
+<polygon width="1.016" layer="1" spacing="1.016" isolate="1.016">
+<vertex x="0" y="127"/>
+<vertex x="88.9" y="127"/>
+<vertex x="88.9" y="0"/>
+<vertex x="0" y="0"/>
+</polygon>
+</signal>
 </signals>
