File: Eagle/Boards/Training Program/UnoMotorShieldsW2016/ISCTrainingProgramw2016_(do first).brd (EAGLE design)
At the start: 89.4 x 131.7 mm, 28 parts, among them J1 ARDUINO_UNO_R3

Commit message: added default board
Parts:
- added E$10: (no value), ISCTRainingProgram:0204/7
- added E$2: (no value), ISCTRainingProgram:RPI-40-HEADER
- added E$3: (no value), ISCTRainingProgram:SN754410NE
- added E$4: (no value), ISCTRainingProgram:5.5-2.5-BARRELCONNECTOR
- added E$5: (no value), ISCTRainingProgram:1X03
- added E$6, E$7: (no value), ISCTRainingProgram:2PIN-SCREW-TERMINAL
- added E$8: (no value), ISCTRainingProgram:E2,5-7
- added E$9: (no value), ISCTRainingProgram:LED5MM
Connections:
- new net S$23: E$5.1
- new net S$24: E$3.P16
- new net S$26: E$2.6, E$8.-
- new net S$27: E$2.33, E$3.P9
- new net S$29: E$2.12
- new net S$30: E$5.3, E$8.+
- new net S$33: E$3.P14
- new net S$35: E$3.P11
- new net S$36: E$3.P7
- new net S$38: E$3.P6
- new net S$39: E$2.7, E$3.P15
- new net S$40: E$2.29
- new net S$41: E$3.P2
- new net S$42: E$3.P8
- new net S$43: E$2.11, E$3.P10
- new net S$46: E$9.K
Routing:
- net S$29: track 0.00 -> 153.2 mm, vias 0 -> 2
- net S$26: track 0.00 -> 86.5 mm, vias 0 -> 1
- net S$24: track 0.00 -> 44.3 mm
- net S$43: track 0.00 -> 43.1 mm, vias 0 -> 1
- net S$33: track 0.00 -> 39.8 mm, vias 0 -> 2
- net S$40: track 0.00 -> 37.6 mm, vias 0 -> 1
- net S$30: track 0.00 -> 37.1 mm, vias 0 -> 2
- net S$35: track 0.00 -> 36.1 mm, vias 0 -> 2
- net S$42: track 0.00 -> 35.9 mm
- net S$36: track 0.00 -> 31.0 mm, vias 0 -> 2
- net S$39: track 0.00 -> 26.3 mm, vias 0 -> 1
- net S$23: track 0.00 -> 21.3 mm, vias 0 -> 1
- net S$27: track 0.00 -> 20.2 mm, vias 0 -> 2
- net S$44: track 0.00 -> 16.7 mm, vias 0 -> 1
- net S$38: track 0.00 -> 16.4 mm, vias 0 -> 1
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- added copper zone on layer 16, net S$28
- added copper zone on layer 1, net S$32
Other:
- outline, holes or cut-outs redrawn
- board text added: "RPi"
