File: Eagle/Boards/Training Program/UnoMotorShieldsW2016/Joseph/EpleyUnoMotorShield.brd (EAGLE design)
At the start: 100 x 80 mm, 5 parts, among them J1 ARDUINO_UNO_R3

Commit message: compiled 1st board for fabrication
Parts:
- added E$1: (no value), ISCTRainingProgram:5.5-2.5-BARRELCONNECTOR
- moved S1 5.59 mm to (18.9, 42.9)
Connections:
- new net S$1: E$1.P$1
- new net S$4: S1.3
- net N$7: no longer S1.3
Routing:
- net S$5: track 0.00 -> 47.7 mm, vias 0 -> 1
- net S$1: track 0.00 -> 36.5 mm, vias 0 -> 1
- net N$7: track 56.3 -> 23.8 mm
- net S$2: track 0.00 -> 11.8 mm
- net S$9: track 0.00 -> 6.35 mm, vias 0 -> 1
- net S$8: track 0.00 -> 6.35 mm, vias 0 -> 1
- net S$7: track 0.00 -> 6.35 mm, vias 0 -> 1
- net S$6: track 0.00 -> 5.08 mm, vias 0 -> 1
- net S$18: track 0.00 -> 5.08 mm, vias 0 -> 1
- net S$21: track 0.00 -> 4.07 mm, vias 0 -> 1
- net S$16: track 0.00 -> 3.18 mm, vias 0 -> 1
- net S$15: track 0.00 -> 3.17 mm, vias 0 -> 1
- net S$14: track 0.00 -> 3.17 mm, vias 0 -> 1
- net S$13: track 0.00 -> 3.17 mm, vias 0 -> 1
- net S$11: track 0.00 -> 3.17 mm
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Other:
- board size 100 x 80 mm -> 64 x 66 mm
Changed lines of the file:
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@@
 <?xml version="1.0" encoding="utf-8"?>
 <!DOCTYPE eagle SYSTEM "eagle.dtd">
-<eagle version="7.2.0">
+<eagle version="7.5.0">
 <drawing>
 <settings>
@@
 <setting verticaltext="up"/>
 </settings>
-<grid distance="0.005" unitdist="inch" unit="inch" style="lines" multiple="1" display="no" altdistance="0.025" altunitdist="inch" altunit="inch"/>
+<grid distance="0.05" unitdist="inch" unit="inch" style="lines" multiple="1" display="no" altdistance="0.025" altunitdist="inch" altunit="inch"/>
 <layers>
 <layer number="1" name="Top" color="4" fill="1" visible="yes" active="yes"/>
+<layer number="2" name="Route2" color="1" fill="3" visible="yes" active="yes"/>
+<layer number="3" name="Route3" color="4" fill="3" visible="yes" active="yes"/>
+<layer number="4" name="Route4" color="1" fill="4" visible="yes" active="yes"/>
+<layer number="5" name="Route5" color="4" fill="4" visible="yes" active="yes"/>
+<layer number="6" name="Route6" color="1" fill="8" visible="yes" active="yes"/>
+<layer number="7" name="Route7" color="4" fill="8" visible="yes" active="yes"/>
+<layer number="8" name="Route8" color="1" fill="2" visible="yes" active="yes"/>
+<layer number="9" name="Route9" color="4" fill="2" visible="yes" active="yes"/>
+<layer number="10" name="Route10" color="1" fill="7" visible="yes" active="yes"/>
+<layer number="11" name="Route11" color="4" fill="7" visible="yes" active="yes"/>
+<layer number="12" name="Route12" color="1" fill="5" visible="yes" active="yes"/>
+<layer number="13" name="Route13" color="4" fill="5" visible="yes" active="yes"/>
+<layer number="14" name="Route14" color="1" fill="6" visible="yes" active="yes"/>
+<layer number="15" name="Route15" color="4" fill="6" visible="yes" active="yes"/>
 <layer number="16" name="Bottom" color="1" fill="1" visible="yes" active="yes"/>
 <layer number="17" name="Pads" color="2" fill="1" visible="yes" active="yes"/>
@@
 <board>
 <plain>
-<wire x1="64" y1="0" x2="100" y2="0" width="0" layer="20"/>
-<wire x1="100" y1="0" x2="100" y2="80" width="0" layer="20"/>
-<wire x1="100" y1="80" x2="0" y2="80" width="0" layer="20"/>
-<wire x1="0" y1="80" x2="0" y2="66" width="0" layer="20"/>
 <wire x1="0" y1="0" x2="0" y2="66" width="1.9304" layer="20"/>
 <wire x1="0" y1="66" x2="64" y2="66" width="1.9304" layer="20"/>
 <wire x1="64" y1="66" x2="64" y2="0" width="1.9304" layer="20"/>
 <wire x1="64" y1="0" x2="0" y2="0" width="1.9304" layer="20"/>
-<text x="19.685" y="55.245" size="3.81" layer="1">JMEPLEY</text>
+<text x="26.035" y="55.245" size="3.81" layer="1">JMEPLEY</text>
 </plain>
 <attributes>
@@
 <elements>
 <element name="J1" library="ISCTRainingProgram" package="ARDUINO_R3" value="ARDUINO_UNO_R3" x="5.27" y="70.55" rot="R270"/>
-<element name="S1" library="ISCTRainingProgram" package="SLIDE_SWITCH" value="" x="18.751" y="48.514"/>
+<element name="S1" library="ISCTRainingProgram" package="SLIDE_SWITCH" value="" x="18.878" y="42.926"/>
 <element name="U$1" library="ISCTRainingProgram" package="DIP16" value="MOTOR_DRIVERDIP16" x="31.73" y="24.9" rot="R270"/>
 <element name="X1" library="ISCTRainingProgram" package="2PIN-SCREW-TERMINAL" value="" x="31.519" y="47.784">
@@
 <attribute name="OC_FARNELL" value="unknown" x="43.616" y="47.784" size="1.778" layer="27" display="off"/>
 </element>
+<element name="E$1" library="ISCTRainingProgram" package="5.5-2.5-BARRELCONNECTOR" value="" x="17.526" y="53.975"/>
 </elements>
 <signals>
@@
 <wire x1="35.54" y1="38.227" x2="35.54" y2="33.79" width="0.8128" layer="16"/>
 </signal>
+<signal name="S$4">
+<contactref element="S1" pad="3"/>
+<wire x1="21.672" y1="42.926" x2="21.59" y2="42.164" width="0.8128" layer="1"/>
+</signal>
 <signal name="N$7">
-<contactref element="S1" pad="3"/>
 <contactref element="J1" pad="VIN"/>
 <contactref element="U$1" pad="P8"/>
@@
 <wire x1="21.59" y1="16.002" x2="27.92" y2="16.002" width="0.8128" layer="1"/>
 <wire x1="27.92" y1="16.002" x2="27.92" y2="16.01" width="0.8128" layer="1"/>
-<wire x1="21.545" y1="48.514" x2="21.59" y2="46.609" width="0.8128" layer="1"/>
-<wire x1="21.59" y1="46.609" x2="21.59" y2="16.002" width="0.8128" layer="1"/>
 </signal>
 <signal name="EN2">
@@
 <contactref element="U$1" pad="P15"/>
 <contactref element="J1" pad="D12"/>
-<wire x1="56.07" y1="39.054" x2="45.593" y2="39.054" width="0.8128" layer="16"/>
-<wire x1="45.593" y1="39.054" x2="41.783" y2="31.242" width="0.8128" layer="16"/>
+<wire x1="56.07" y1="39.054" x2="45.593" y2="37.784" width="0.8128" layer="16"/>
+<wire x1="45.593" y1="37.784" x2="41.783" y2="31.242" width="0.8128" layer="16"/>
 <wire x1="41.783" y1="31.242" x2="35.54" y2="31.242" width="0.8128" layer="16"/>
 <wire x1="35.54" y1="31.242" x2="35.54" y2="31.25" width="0.8128" layer="16"/>
 </signal>
+<signal name="S$1">
+<wire x1="7.874" y1="29.972" x2="10.922" y2="29.972" width="1.9304" layer="1"/>
+<wire x1="10.922" y1="29.972" x2="12.065" y2="29.845" width="1.9304" layer="1"/>
+<contactref element="E$1" pad="P$1"/>
+<wire x1="12.065" y1="29.845" x2="12.065" y2="47.371" width="1.9304" layer="1"/>
+<wire x1="12.065" y1="47.371" x2="12.065" y2="50.292" width="1.9304" layer="1"/>
+<wire x1="12.065" y1="50.292" x2="14.478" y2="53.975" width="1.9304" layer="1"/>
+<wire x1="14.478" y1="53.975" x2="12.065" y2="50.292" width="1.9304" layer="16"/>
+<wire x1="12.065" y1="50.292" x2="12.065" y2="47.371" width="1.9304" layer="16"/>
+<wire x1="12.065" y1="47.371" x2="12.065" y2="47.244" width="1.9304" layer="16"/>
+<via x="12.065" y="47.371" extent="1-16" drill="0.6"/>
+</signal>
+<signal name="S$2">
+<wire x1="20.574" y1="53.848" x2="20.574" y2="52.197" width="1.9304" layer="16"/>
+<wire x1="20.574" y1="52.197" x2="21.717" y2="51.054" width="1.9304" layer="16"/>
+<wire x1="21.717" y1="51.054" x2="21.717" y2="42.545" width="1.9304" layer="16"/>
+</signal>
+<signal name="S$3">
+<via x="18.796" y="39.624" extent="1-16" drill="0.6"/>
+</signal>
+<signal name="S$5">
+<wire x1="18.923" y1="42.926" x2="18.923" y2="29.972" width="1.9304" layer="1"/>
+<wire x1="18.923" y1="29.972" x2="13.843" y2="24.892" width="1.9304" layer="1"/>
+<wire x1="13.843" y1="24.892" x2="12.954" y2="24.892" width="1.9304" layer="1"/>
+<wire x1="7.874" y1="24.892" x2="12.954" y2="24.892" width="1.9304" layer="1"/>
+<wire x1="12.954" y1="24.892" x2="21.971" y2="15.875" width="1.9304" layer="1"/>
+<wire x1="21.971" y1="15.875" x2="25.4" y2="15.875" width="1.9304" layer="1"/>
+<wire x1="25.4" y1="15.875" x2="28.321" y2="15.875" width="1.9304" layer="1"/>
+<via x="25.4" y="15.875" extent="1-16" drill="0.6"/>
+<wire x1="25.4" y1="15.875" x2="27.94" y2="15.875" width="1.016" layer="16"/>
+</signal>
+<signal name="S$6">
+<wire x1="29.21" y1="45.72" x2="29.21" y2="40.64" width="1.9304" layer="16"/>
+<via x="29.21" y="40.64" extent="1-16" drill="0.6"/>
+</signal>
+<signal name="S$7">
+<wire x1="34.29" y1="46.99" x2="34.29" y2="40.64" width="1.9304" layer="16"/>
+<via x="34.29" y="40.64" extent="1-16" drill="0.6"/>
+</signal>
+<signal name="S$8">
+<wire x1="40.64" y1="46.99" x2="40.64" y2="40.64" width="1.9304" layer="16"/>
+<via x="40.64" y="40.64" extent="1-16" drill="0.6"/>
+</signal>
+<signal name="S$9">
+<wire x1="45.72" y1="46.99" x2="45.72" y2="40.64" width="1.9304" layer="16"/>
+<via x="45.72" y="40.64" extent="1-16" drill="0.6"/>
+</signal>
+<signal name="S$10">
+<via x="10.16" y="33.02" extent="1-16" drill="0.6"/>
+<wire x1="7.62" y1="32.385" x2="9.525" y2="32.385" width="1.016" layer="1"/>
+<wire x1="9.525" y1="32.385" x2="10.16" y2="33.02" width="1.016" layer="1"/>
+</signal>
+<signal name="S$11">
+<wire x1="19.05" y1="40.005" x2="19.05" y2="43.18" width="1.016" layer="16"/>
+</signal>
+<signal name="S$12">
+<via x="38.1" y="28.575" extent="1-16" drill="0.6"/>
+<wire x1="36.195" y1="28.575" x2="38.1" y2="28.575" width="1.016" layer="16"/>
+</signal>
+<signal name="S$13">
+<via x="38.735" y="20.955" extent="1-16" drill="0.6"/>
+<wire x1="35.56" y1="20.955" x2="38.735" y2="20.955" width="1.016" layer="16"/>
+</signal>
+<signal name="S$14">
+<via x="38.735" y="18.415" extent="1-16" drill="0.6"/>
+<wire x1="35.56" y1="18.415" x2="38.735" y2="18.415" width="1.016" layer="16"/>
+</signal>
+<signal name="S$15">
+<via x="38.735" y="15.875" extent="1-16" drill="0.6"/>
+<wire x1="35.56" y1="15.875" x2="38.735" y2="15.875" width="1.016" layer="16"/>
+</signal>
+<signal name="S$16">
+<via x="24.765" y="20.955" extent="1-16" drill="0.6"/>
+<wire x1="24.765" y1="20.955" x2="27.94" y2="20.955" width="1.016" layer="16"/>
+</signal>
+<signal name="S$17">
+<via x="25.4" y="28.575" extent="1-16" drill="0.6"/>
+<wire x1="25.4" y1="28.575" x2="27.94" y2="28.575" width="1.016" layer="16"/>
+</signal>
+<signal name="S$18">
+<via x="38.1" y="25.4" extent="1-16" drill="0.6"/>
+<wire x1="35.56" y1="25.4" x2="38.1" y2="25.4" width="1.016" layer="16"/>
+<wire x1="35.56" y1="25.4" x2="38.1" y2="25.4" width="1.016" layer="1"/>
+</signal>
+<signal name="S$19">
+<via x="53.34" y="39.37" extent="1-16" drill="0.6"/>
+<wire x1="53.34" y1="39.37" x2="55.88" y2="39.37" width="1.016" layer="1"/>
+</signal>
+<signal name="S$20">
+<via x="53.34" y="29.21" extent="1-16" drill="0.6"/>
+<wire x1="53.34" y1="29.21" x2="55.88" y2="29.21" width="1.016" layer="1"/>
+</signal>
+<signal name="S$21">
+<via x="52.07" y="24.13" extent="1-16" drill="0.6"/>
+<wire x1="52.07" y1="24.13" x2="53.34" y2="24.13" width="1.016" layer="1"/>
+<wire x1="53.34" y1="24.13" x2="53.975" y2="24.765" width="1.016" layer="1"/>
+<wire x1="53.975" y1="24.765" x2="55.88" y2="24.765" width="1.016" layer="1"/>
+</signal>
+<signal name="S$22">
+<via x="53.34" y="21.59" extent="1-16" drill="0.6"/>
+<wire x1="53.34" y1="21.59" x2="53.975" y2="22.225" width="1.016" layer="1"/>
+<wire x1="53.975" y1="22.225" x2="55.88" y2="22.225" width="1.016" layer="1"/>
+</signal>
 </signals>

Commit message: updated Joseph's board
Parts:
- added JP1, JP2: (no value), ISCTRainingProgram:1X03
- moved E$1 3.72 mm to (17.0, 50.3)
- moved S1 3.61 mm to (17.7, 39.5)
- moved X1 1.40 mm to (30.1, 47.9)
- moved X2 1.40 mm to (45.0, 47.8)
Connections:
- removed net S$1: E$1.P$1
- removed net S$4: S1.3
- new net N$11: J1.D4, JP1.1
- new net N$12: J1.5V, JP1.2, JP2.2, U$1.P16
- net GND: now also JP1.3, JP2.3
- net N$5: now also J1.D2, JP2.1; no longer J1.5V, U$1.P16
- net N$7: now also S1.3
Routing:
- net N$12: track 0.00 -> 73.6 mm
- net N$11: track 0.00 -> 54.9 mm
- net GND: track 36.0 -> 90.4 mm
- net S$5: track 47.7 -> 0.00 mm, vias 1 -> 0
- net N$5: track 34.6 -> 79.1 mm
- net N$7: track 23.8 -> 47.9 mm
- net S$1: track 36.5 -> 23.3 mm, vias 1 -> 0
- net S$3: track 0.00 -> 9.94 mm, vias 1 -> 0
- net S$9: track 6.35 -> 0.00 mm, vias 1 -> 0
- net S$8: track 6.35 -> 0.00 mm, vias 1 -> 0
- net S$7: track 6.35 -> 0.00 mm, vias 1 -> 0
- net S$6: track 5.08 -> 0.00 mm, vias 1 -> 0
- net S$18: track 5.08 -> 0.00 mm, vias 1 -> 0
- net S$21: track 4.07 -> 0.00 mm, vias 1 -> 0
- net S$16: track 3.18 -> 0.00 mm, vias 1 -> 0
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- added copper zone on layer 16, net S$4
- added copper zone on layer 1, net S$5
